File: KiCad/C3/Unified-Daughterboard.kicad_pcb (KiCad board)
At the start: 2 copper layers, 18 x 16.5 mm, 18 parts, among them IC1 NCP380LSN05AAT1G, J1 TYPE-C-31-M12_13, J2 SM04B-SRSS-TB(LF)(SN), J3 Conn_02x02_Odd_Even, U1 TPD4E05U06DQAR

Commit message: some changes
Parts:
- removed G1: Unified-Daughterboard-Logo, Unified-Daughterboard-Logo:Unified-Daughterboard-Logo.pretty
