File: KiCad/C3/Unified-Daughterboard.kicad_sch (KiCad schematic)
At the start: 18 parts, among them IC1 NCP380LSN05AAT1G, J1 TYPE-C-31-M12_13, J2 SM04B-SRSS-TB(LF)(SN), U1 TPD4E05U06DQAR

Commit message: some changes
Parts:
- removed G1: Unified-Daughterboard-Logo, Unified-Daughterboard-Logo:Unified-Daughterboard-Logo.pretty, symbol Mechanical:MountingHole
Changed lines of the file:
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@@
     (pin "2")
-  )
-  (symbol (lib_id "Mechanical:MountingHole") (at 234.315 53.34 0) (unit 1)
-    (in_bom yes) (on_board yes)
-    (property "Reference" "G1" (id 0) (at 236.855 52.197 0)
-      (effects (font (size 1.27 1.27)) (justify left))
-    )
-    (property "Value" "Unified-Daughterboard-Logo" (id 1) (at 236.855 54.483 0)
-      (effects (font (size 1.27 1.27)) (justify left))
-    )
-    (property "Footprint" "Unified-Daughterboard-Logo:Unified-Daughterboard-Logo.pretty" (id 2) (at 234.315 53.34 0)
-      (effects (font (size 1.27 1.27)) hide)
-    )
-    (property "Datasheet" "~" (id 3) (at 234.315 53.34 0)
-      (effects (font (size 1.27 1.27)) hide)
-    )
   )
   (symbol (lib_id "power:GNDPWR") (at 32.385 119.38 0) (unit 1)
@@
       (reference "F1") (unit 1) (value "ASMD1206-150") (footprint "Fuse:Fuse_0603_1608Metric_Pad1.05x0.95mm_HandSolder")
     )
-    (path "/00000000-0000-0000-0000-00005e790861"
-      (reference "G1") (unit 1) (value "Unified-Daughterboard-Logo") (footprint "Unified-Daughterboard-Logo:Unified-Daughterboard-Logo.pretty")
-    )
     (path "/00000000-0000-0000-0000-00005e780029"

Commit message: change back and add decoupling cap
Parts:
- removed IC1: NCP380LSN05AAT1G, SamacSys_Parts:SOT95P275X110-5N, symbol SamacSys_Parts:NCP380LSN05AAT1G
- removed MH1, MH2, MH3, MH4: Mount-M2, random-keyboard-parts:Generic-Mounthole, symbol Connector_Generic:Conn_01x01
- removed R3: 100k, Resistor_SMD:R_0402_1005Metric_Pad0.72x0.64mm_HandSolder, symbol Device:R_Small
- added H1, H2, H3, H4: MountingHole_Pad, MountingHole:MountingHole_2.2mm_M2_DIN965_Pad_TopBottom, symbol Mechanical:MountingHole_Pad
- C1: value 1u -> 10u; footprint (none) -> Capacitor_SMD:C_0805_2012Metric
- D1: footprint acheron_Components:D_SOD-123_Bidirectional -> Diode_SMD:D_SOD-123
- J3: value (none) -> Conn_02x02_Odd_Even; footprint (none) -> Connector_PinHeader_1.27mm:PinHeader_2x02_P1.27mm_Horizontal
Connections:
- net VCCQ is gone; now on net VCC: J2.1 (Pin_1), J3.4 (Pin_4)
- net GNDPWR: now also H1.1, H2.1, H3.1, H4.1; no longer C1.2, D1.1 (A1), J1.A1 (GND), J1.B1 (GND), L1.2, R1.2, R2.2, U1.3 (GND), U1.8 (GND)
- net VBUS: now also C1.1
- net VCC: no longer C1.1
- new net GNDREF: C1.2, D1.1 (A1), J1.A1 (GND), J1.B1 (GND), L1.2, R1.2, R2.2, U1.3 (GND), U1.8 (GND)
Other:
- moved on the sheet: D1, F1
